File: candle-lamp.kicad_sch (KiCad schematic)
At the start: 11 parts

Commit message: upd
Parts:
- removed R?: R, symbol Device:R
- removed R?: R_Variable, symbol Device:R_Variable
- added R?: R, symbol Device:R
- added R?: R_Variable, symbol Device:R_Variable
Connections:
- net GND: now also R?.2
- net VDD: now also R?.1
- net Vref: now also R?.1, R?.2
Other:
- note added: "How to spec this? Largest serial resistance possible to min. wasted power Vref = Vdd * R_variable / (R + R_variable)"
- note removed: "How to spec this? Largest serial resistance possible to min. wasted power"
Changed lines of the file:
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@@
     (effects (font (size 5 5)) (justify left bottom))
   )
-  (text "Generator" (at 24.13 30.48 0)
+  (text "Generator" (at 24.13 31.75 0)
     (effects (font (size 5 5)) (justify left bottom))
   )
-  (text "How to spec this?\nLargest serial resistance possible to min. wasted power"
-    (at 201.93 80.01 0)
+  (text "How to spec this?\nLargest serial resistance possible to min. wasted power\n\nVref = Vdd * R_variable / (R + R_variable)"
+    (at 201.93 83.82 0)
     (effects (font (size 1.27 1.27)) (justify left bottom))
   )
@@
     )
   )
+  (symbol (lib_id "Device:R") (at 226.06 48.26 0) (unit 1)
+    (in_bom yes) (on_board yes) (fields_autoplaced)
+    (property "Reference" "R?" (id 0) (at 228.6 46.9899 0)
+      (effects (font (size 1.27 1.27)) (justify left))
+    )
+    (property "Value" "R" (id 1) (at 228.6 49.5299 0)
+      (effects (font (size 1.27 1.27)) (justify left))
+    )
+    (property "Footprint" "" (id 2) (at 224.282 48.26 90)
+      (effects (font (size 1.27 1.27)) hide)
+    )
+    (property "Datasheet" "~" (id 3) (at 226.06 48.26 0)
+      (effects (font (size 1.27 1.27)) hide)
+    )
+    (pin "1")
+    (pin "2")
+  )
   (symbol (lib_id "Device:Lamp") (at 129.54 160.02 0) (unit 1)
     (in_bom yes) (on_board yes) (fields_autoplaced)
@@
     )
     (pin "1")
-  )
-  (symbol (lib_id "Device:R") (at 226.06 63.5 0) (unit 1)
-    (in_bom yes) (on_board yes) (fields_autoplaced)
-    (property "Reference" "R?" (id 0) (at 228.6 62.2299 0)
-      (effects (font (size 1.27 1.27)) (justify left))
-    )
-    (property "Value" "R" (id 1) (at 228.6 64.7699 0)
-      (effects (font (size 1.27 1.27)) (justify left))
-    )
-    (property "Footprint" "" (id 2) (at 224.282 63.5 90)
-      (effects (font (size 1.27 1.27)) hide)
-    )
-    (property "Datasheet" "~" (id 3) (at 226.06 63.5 0)
-      (effects (font (size 1.27 1.27)) hide)
-    )
-    (pin "1")
-    (pin "2")
   )
   (symbol (lib_id "power:VDD") (at 41.91 138.43 0) (unit 1)
@@
     (pin "3")
   )
-  (symbol (lib_id "Device:R_Variable") (at 226.06 48.26 0) (unit 1)
-    (in_bom yes) (on_board yes) (fields_autoplaced)
-    (property "Reference" "R?" (id 0) (at 229.87 46.9899 0)
-      (effects (font (size 1.27 1.27)) (justify left))
-    )
-    (property "Value" "R_Variable" (id 1) (at 229.87 49.5299 0)
-      (effects (font (size 1.27 1.27)) (justify left))
-    )
-    (property "Footprint" "" (id 2) (at 224.282 48.26 90)
-      (effects (font (size 1.27 1.27)) hide)
-    )
-    (property "Datasheet" "~" (id 3) (at 226.06 48.26 0)
-      (effects (font (size 1.27 1.27)) hide)
-    )
-    (pin "1")
-    (pin "2")
-  )
   (symbol (lib_id "power:GND") (at 149.86 74.93 0) (unit 1)
     (in_bom yes) (on_board yes) (fields_autoplaced)
@@
     )
     (property "Datasheet" "~" (id 3) (at 22.86 53.086 0)
+      (effects (font (size 1.27 1.27)) hide)
+    )
+    (pin "1")
+    (pin "2")
+  )
+  (symbol (lib_id "Device:R_Variable") (at 226.06 63.5 0) (unit 1)
+    (in_bom yes) (on_board yes) (fields_autoplaced)
+    (property "Reference" "R?" (id 0) (at 229.87 62.2299 0)
+      (effects (font (size 1.27 1.27)) (justify left))
+    )
+    (property "Value" "R_Variable" (id 1) (at 229.87 64.7699 0)
+      (effects (font (size 1.27 1.27)) (justify left))
+    )
+    (property "Footprint" "" (id 2) (at 224.282 63.5 90)
+      (effects (font (size 1.27 1.27)) hide)
+    )
+    (property "Datasheet" "~" (id 3) (at 226.06 63.5 0)
       (effects (font (size 1.27 1.27)) hide)
     )
@@
       (reference "Q?") (unit 1) (value "2N7000") (footprint "Package_TO_SOT_THT:TO-92_Inline")
     )
-    (path "/3ad319dd-a8ca-495c-bb4c-a4f646618f3d"
+    (path "/0289a5ff-c156-4137-9c4a-d65d6d4d4a77"
       (reference "R?") (unit 1) (value "R") (footprint "")
     )
@@
       (reference "R?") (unit 1) (value "R Pullup") (footprint "")
     )
-    (path "/902029bc-6174-48c7-b1cd-cdc91135507c"
+    (path "/bd61f932-e93d-45ab-a0d6-8f63e9f955c8"
       (reference "R?") (unit 1) (value "R_Variable") (footprint "")
     )
