File: candle-lamp.kicad_sch (KiCad schematic)
At the start: 11 parts, among them M1 Fan

Commit message: leaky-opamp
Parts:
- removed C1: 10 nF, symbol pspice:CAP
- removed LA?: Lamp!, symbol Device:Lamp
- removed R1: 5.1 MΩ, symbol Device:R
- added Cint: C?, symbol Device:C
- added LA?: Lamp!, symbol Device:Lamp
- added Rdrain, Rfan: R, symbol Device:R
- added U: TLV9062xD, Package_SO:SOIC-8_3.9x4.9mm_P1.27mm, symbol Amplifier_Operational:TLV9062xD
Connections:
- net +12V: now also LA?.2 (+); no longer Q?.3 (D)
- net GND: now also Q?.1 (S), U.3 (+)
- net Vout, Fan: now also Cint.2, Rdrain.1, U.1; no longer M1.1 (+)
- new net: M1.1 (+), Rfan.1
- new net: Cint.1, Rdrain.2, Rfan.2, U.2 (-)
- new net: LA?.1 (-), Q?.3 (D)
Other:
- note added: "TODO: - spec. transistor (https://www.digikey.com/short/0tzzmv54) - spec high voltage - what light? - 2N7000 has max Id = 200 mA. Need stronger transistor - Relay instead???"
- note removed: "TODO: - figure out req'd voltages for mosfet - spec. transistor - spec high voltage"
- note removed: "What time constant do we want here? For the RPi fan, we get a very noisy signal that needs to be smoothed. There is probably some better way to do this. Mabye OpAmp integrator circuit? We also have to amplify this. With the RC constants chosen here, we get ~250 - 500 mV, with 250 mV stable and 250 - 500 mV of noise. If we amplify by a factor of 5, we get 1.25 V to 2.5 V. We can set Vref to ~0.8 V."
- moved on the sheet: M1, Q?
